Commit message: fix(urdf): update mesh refs to match renamed xela_models files
ft_c.stl → uSCuAH.stl, 4x4.stl → uSPa44.stl following the rename
in xela_models commit 893f77b (xacro file refactoring, 2026-02-12).

Co-Authored-By: Claude Sonnet 4.6 <noreply@anthropic.com>

File: xela_ah_r2c_bringup/urdf/x_allegro_left_no_taxel.urdf (robot description, URDF)
Before this commit: robot allegro_hand_left, 45 links, 44 joints
Links:
- link base_x_taxel_0_01_4x4_link: geometry collision mesh filename=package://xela_models/mesh/uSPa44.stl; visual mesh filename=package://xela_models/mesh/uSPa44.stl
- link base_x_taxel_0_02_4x4_link: geometry collision mesh filename=package://xela_models/mesh/uSPa44.stl; visual mesh filename=package://xela_models/mesh/uSPa44.stl
- link base_x_taxel_0_03_aftc_link: geometry collision mesh filename=package://xela_models/mesh/uSCuAH.stl; visual mesh filename=package://xela_models/mesh/uSCuAH.stl scale=0.93 0.93 0.93
- link base_x_taxel_0_10_4x4_link: geometry collision mesh filename=package://xela_models/mesh/uSPa44.stl; visual mesh filename=package://xela_models/mesh/uSPa44.stl
- link base_x_taxel_0_11_4x4_link: geometry collision mesh filename=package://xela_models/mesh/uSPa44.stl; visual mesh filename=package://xela_models/mesh/uSPa44.stl
- link base_x_taxel_0_12_4x4_link: geometry collision mesh filename=package://xela_models/mesh/uSPa44.stl; visual mesh filename=package://xela_models/mesh/uSPa44.stl
- link base_x_taxel_0_13_aftc_link: geometry collision mesh filename=package://xela_models/mesh/uSCuAH.stl; visual mesh filename=package://xela_models/mesh/uSCuAH.stl scale=0.93 0.93 0.93
- link base_x_taxel_0_20_4x4_link: geometry collision mesh filename=package://xela_models/mesh/uSPa44.stl; visual mesh filename=package://xela_models/mesh/uSPa44.stl
- link base_x_taxel_0_21_4x4_link: geometry collision mesh filename=package://xela_models/mesh/uSPa44.stl; visual mesh filename=package://xela_models/mesh/uSPa44.stl
- link base_x_taxel_0_22_4x4_link: geometry collision mesh filename=package://xela_models/mesh/uSPa44.stl; visual mesh filename=package://xela_models/mesh/uSPa44.stl
- link base_x_taxel_0_23_aftc_link: geometry collision mesh filename=package://xela_models/mesh/uSCuAH.stl; visual mesh filename=package://xela_models/mesh/uSCuAH.stl scale=0.93 0.93 0.93
- link base_x_taxel_0_30_4x4_link: geometry collision mesh filename=package://xela_models/mesh/uSPa44.stl; visual mesh filename=package://xela_models/mesh/uSPa44.stl
- link base_x_taxel_0_31_4x4_link: geometry collision mesh filename=package://xela_models/mesh/uSPa44.stl; visual mesh filename=package://xela_models/mesh/uSPa44.stl
- link base_x_taxel_0_32_4x4_link: geometry collision mesh filename=package://xela_models/mesh/uSPa44.stl; visual mesh filename=package://xela_models/mesh/uSPa44.stl
- link base_x_taxel_0_33_aftc_link: geometry collision mesh filename=package://xela_models/mesh/uSCuAH.stl; visual mesh filename=package://xela_models/mesh/uSCuAH.stl scale=0.93 0.93 0.93
