Commit message: update xacro

File: xela_ah_r2c_bringup/urdf/allegro_hand_left_r2c.xacro (robot description, xacro)
@@ -508,5 +508,5 @@
     <joint name="ah_joint${finger_num}1" type="revolute">
       <axis xyz="0 0 -1"/>
-      <limit effort="15" velocity="7" lower="${-0.205+0.1}" upper="${1.263-0.1}" />
+      <limit effort="15" velocity="7" lower="${-0.30}" upper="${1.263-0.1}" />
       <parent link="${sequence}ah_link_${finger_num}0"/>
       <child link="${sequence}ah_link_${finger_num}1"/>

File: xela_ah_r2c_bringup/urdf/allegro_hand_right_r2c.xacro (robot description, xacro)
@@ -304,5 +304,5 @@
       </xacro:if>
       <joint name="ah_joint${finger_num}1" type="revolute">
-        <limit effort="15" velocity="7" lower="${-0.296+0.1}" upper="${1.71-0.1}" />
+        <limit effort="15" velocity="7" lower="${-0.296+0.1}" upper="1.75" />
         <axis xyz="0 1 0"/>
         <parent link="${sequence}ah_link_${finger_num}0"/>
@@ -460,5 +460,5 @@
     <joint name="ah_joint${finger_num}0" type="revolute">
       <axis xyz="-1 0 0"/>
-      <limit effort="15" velocity="7" lower="${0.363-0.1}" upper="${1.496-0.1}" />
+      <limit effort="15" velocity="7" lower="${0.363-0.1}" upper="1.55" />
       <parent link="${parent}"/>
       <child link="${sequence}ah_link_${finger_num}0"/>
