Commit message: joint limt update

File: xela_ah_r2c_bringup/urdf/allegro_hand_right_r2c.xacro (robot description, xacro)
@@ -508,5 +508,5 @@
     <joint name="ah_joint${finger_num}1" type="revolute">
       <axis xyz="0 0 1"/>
-      <limit effort="15" velocity="7" lower="${-0.205+0.1}" upper="${1.263-0.1}" />
+      <limit effort="15" velocity="7" lower="${-0.30}" upper="${1.263-0.1}" />
       <parent link="${sequence}ah_link_${finger_num}0"/>
       <child link="${sequence}ah_link_${finger_num}1"/>

Commit message: Fix: Update allegro hand right r2c XACRO configuration

File: xela_ah_r2c_bringup/urdf/allegro_hand_right_r2c.xacro (robot description, xacro)
@@ -582,5 +582,5 @@
     <joint name="ah_joint${finger_num}2" type="revolute">
       <axis xyz="0 1 0"/>
-      <limit effort="15" velocity="7" lower="${-0.289+0.1}" upper="${1.744-0.1}" />
+      <limit effort="15" velocity="7" lower="${-0.289}" upper="${1.744-0.1}" />
       <parent link="${sequence}ah_link_${finger_num}1"/>
       <child link="${sequence}ah_link_${finger_num}2"/>
